Commit message: Update robot-ackerman.urdf

File: robot-ackerman.urdf (robot description, URDF)
Before this commit: robot roboto, 9 links, 8 joints
Links:
- link base_link: mass 20.0 -> 5.0; geometry collision box size=0.5 0.25 0.1; visual box size=0.5 0.25 0.1
- link front_left_axle: geometry collision box size=0.1 0.1 0.1; visual box size=0.1 0.1 0.1
- link front_left_wheel: geometry collision cylinder length=0.1 radius=0.08; visual cylinder length=0.1 radius=0.08
- link front_right_axle: geometry collision box size=0.1 0.1 0.1; visual box size=0.1 0.1 0.1
- link front_right_wheel: geometry collision cylinder length=0.1 radius=0.08; visual cylinder length=0.1 radius=0.08
- link rear_left_axle: geometry collision box size=0.1 0.1 0.1; visual box size=0.1 0.1 0.1
- link rear_left_wheel: geometry collision cylinder length=0.1 radius=0.08; visual cylinder length=0.1 radius=0.08
- link rear_right_axle: geometry collision box size=0.1 0.1 0.1; visual box size=0.1 0.1 0.1
- link rear_right_wheel: geometry collision cylinder length=0.1 radius=0.08; visual cylinder length=0.1 radius=0.08
